Commit message: fix mesh address in urdf

File: src/my_second_robot/urdf/robot_w_screwdriver.urdf (robot description, URDF)
Before this commit: robot irb6640_205, 13 links, 12 joints
Links:
- link base_link: geometry collision mesh filename=package://my_second_robot/meshes/irb6640_205/base_link.dae; visual mesh filename=package://my_second_robot/meshes/irb6640_205/base_link.dae
- link cylinder_link: geometry collision mesh filename=package://my_second_robot/meshes/irb6640_205/cylinder_link.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; visual mesh filename=package://my_second_robot/meshes/irb6640_205/cylinder_link.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
- link link1: geometry collision mesh filename=package://my_second_robot/meshes/irb6640_205/link1.dae; visual mesh filename=package://my_second_robot/meshes/irb6640_205/link1.dae
- link link2: geometry collision mesh filename=package://my_second_robot/meshes/irb6640_205/link2.dae; visual mesh filename=package://my_second_robot/meshes/irb6640_205/link2.dae
- link link3: geometry collision mesh filename=package://my_second_robot/meshes/irb6640_205/link3.dae; visual mesh filename=package://my_second_robot/meshes/irb6640_205/link3.dae
- link link4: geometry collision mesh filename=package://my_second_robot/meshes/irb6640_205/link4.dae; visual mesh filename=package://my_second_robot/meshes/irb6640_205/link4.dae
- link link5: geometry collision mesh filename=package://my_second_robot/meshes/irb6640_205/link5.dae; visual mesh filename=package://my_second_robot/meshes/irb6640_205/link5.dae
- link link6: geometry collision mesh filename=package://my_second_robot/meshes/irb6640_205/link6.dae; visual mesh filename=package://my_second_robot/meshes/irb6640_205/link6.dae
- link piston_link: geometry collision mesh filename=package://my_second_robot/meshes/irb6640_205/piston_link.dae; visual mesh filename=package://my_second_robot/meshes/irb6640_205/piston_link.dae
- link screwdriver: geometry collision mesh filename=package://my_second_robot/meshes/screwdriver/weber_screwdri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; visual mesh filename=package://my_second_robot/meshes/screwdriver/weber_screwdri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

Commit message: add screw and box to gazebo

File: src/my_second_robot/urdf/robot_w_screwdriver.urdf (robot description, URDF)
Before this commit: robot my_second_robot, 13 links, 12 joints
Links:
- removed link base
