Commit message: load both robot and screw in gazebo

File: src/my_second_robot/urdf/assembly.xacro (robot description, xacro)
@@ -1,28 +1,23 @@
 <?xml version="1.0" ?>
 <robot xmlns:xacro="http://www.ros.org/wiki/xacro" name="assembly">
-  <link name="base">
-        <visual>
-            <geometry>
-                <box size="0.1 0.1 0.01"/> <!-- Small base plate -->
-            </geometry>
-            <material name="gray">
-                <color rgba="0.5 0.5 0.5 1"/>
-            </material>
-        </visual>
-        <collision>
-            <geometry>
-                <box size="0.1 0.1 0.01"/>
-            </geometry>
-        </collision>
-        <inertial>
-            <mass value="0.1"/>
-            <inertia ixx="0.001" iyy="0.001" izz="0.001" ixy="0" ixz="0" iyz="0"/>
-        </inertial>
-    </link>
+  <!-- Base link -->
+<link name="base"/>
+  <!-- Explicitly fix base to Gazebo world -->
+  <gazebo reference="base">
+    <static>true</static>
+  </gazebo>
   <!-- Include my_second_robot -->
-  <xacro:include filename="$(find my_second_robot)/urdf/robot_in_gz.urdf"/>
-  <!-- <xacro:robot_w_screwdriver/> -->
+  <xacro:include filename="$(find my_second_robot)/urdf/robot.urdf"/>
+  <joint name="robot_joint" type="fixed">
+    <parent link="base"/>
+    <child link="base_link"/>
+    <origin xyz="2 0 -0.5" rpy="0 0 3.14"/>
+  </joint>
   <!-- Include screw_model -->
-  <xacro:include filename="$(find my_second_robot)/urdf/screws_in_gz.urdf"/>
-  <!-- <xacro:screws/> -->
+  <xacro:include filename="$(find my_second_robot)/urdf/screws.urdf"/>
+  <joint name="screws_joint" type="fixed">
+    <parent link="base"/>
+    <child link="box"/>
+    <origin xyz="0 0 0.01" rpy="0 0 0"/>
+  </joint>
 </robot>

File: src/my_second_robot/urdf/robot.urdf (robot description, URDF)
Before this commit: robot my_second_robot, 13 links, 12 joints
Links:
- removed link base
Joints:
- removed joint base_link-base

File: src/my_second_robot/urdf/screws.urdf (robot description, URDF)
Before this commit: robot screws, 3 links, 2 joints
Links:
- removed link base
Joints:
- removed joint box_joint

Commit message: use cart_position example to load gz_ros2 package

File: src/my_second_robot/urdf/assembly.xacro (robot description, xacro)
@@ -1,23 +1,32 @@
 <?xml version="1.0" ?>
 <robot xmlns:xacro="http://www.ros.org/wiki/xacro" name="assembly">
-  <!-- Base link -->
-<link name="base"/>
-  <!-- Explicitly fix base to Gazebo world -->
-  <gazebo reference="base">
-    <static>true</static>
-  </gazebo>
+<link name="world"/>
+  <!-- Base link shared by all -->
+  <link name="base">
+    <inertial>
+      <mass value="1.0"/>
+      <origin xyz="0 0 0"/>
+      <inertia ixx="1e-6" ixy="0.0" ixz="0.0" iyy="1e-6" iyz="0.0" izz="1e-6"/>
+    </inertial>
+  </link>
+    <!-- Fix base_link to the Gazebo world -->
+  <joint name="base_fixed_to_world" type="fixed">
+    <parent link="world"/>
+    <child link="base"/>
+    <origin xyz="0 0 0" rpy="0 0 0"/>
+  </joint>
   <!-- Include my_second_robot -->
   <xacro:include filename="$(find my_second_robot)/urdf/robot.urdf"/>
-  <joint name="robot_joint" type="fixed">
+  <joint name="robot_to_base" type="fixed">
     <parent link="base"/>
     <child link="base_link"/>
-    <origin xyz="2 0 -0.5" rpy="0 0 3.14"/>
+    <origin xyz="2 0 0" rpy="0 0 3.14"/>
   </joint>
   <!-- Include screw_model -->
   <xacro:include filename="$(find my_second_robot)/urdf/screws.urdf"/>
-  <joint name="screws_joint" type="fixed">
+  <joint name="box_to_base" type="fixed">
     <parent link="base"/>
     <child link="box"/>
-    <origin xyz="0 0 0.01" rpy="0 0 0"/>
+    <origin xyz="0 0 0.5" rpy="0 0 0"/>
   </joint>
   <!-- Gazebo Plugin for ros2_control -->
