Commit message: fix the zero effort in robot urdf

File: src/my_second_robot/urdf/robot.urdf (robot description, URDF)
Before this commit: robot my_second_robot, 12 links, 11 joints
Joints:
- joint joint_1: limit lower=-2.9670597283903604 upper=2.9670597283903604 effort=0 velocity=1.7453292519943295 -> lower=-2.9670597283903604 upper=2.9670597283903604 effort=10 velocity=1.7453292519943295
- joint joint_2: limit lower=-1.1344640137963142 upper=1.4835298641951802 effort=0 velocity=1.5707963267948966 -> lower=-1.1344640137963142 upper=1.4835298641951802 effort=10 velocity=1.5707963267948966
- joint joint_3: limit lower=-3.141592653589793 upper=1.2217304763960306 effort=0 velocity=1.5707963267948966 -> lower=-3.141592653589793 upper=1.2217304763960306 effort=10 velocity=1.5707963267948966
- joint joint_4: limit lower=-5.235987755982989 upper=5.235987755982989 effort=0 velocity=2.9670597283903604 -> lower=-5.235987755982989 upper=5.235987755982989 effort=10 velocity=2.9670597283903604
- joint joint_5: limit lower=-1.7453292519943295 upper=1.7453292519943295 effort=0 velocity=2.0943951023931953 -> lower=-1.7453292519943295 upper=1.7453292519943295 effort=10 velocity=2.0943951023931953
- joint joint_6: limit lower=-6.283185307179586 upper=6.283185307179586 effort=0 velocity=3.3161255787892263 -> lower=-6.283185307179586 upper=6.283185307179586 effort=10 velocity=3.3161255787892263
