Commit message: add multiple screws

File: src/moving6/urdf/circu_screws.urdf (robot description, URDF)
Before this commit: robot screws, 2 links, 1 joints
Links:
- removed link screw_torx_T30
- added link screw_0, mass 0.002; collision cylinder length=0.03 radius=0.015; visual cylinder length=0.03 radius=0.015
- added link screw_1, mass 0.002; collision cylinder length=0.03 radius=0.015; visual cylinder length=0.03 radius=0.015
- added link screw_2, mass 0.002; collision cylinder length=0.03 radius=0.015; visual cylinder length=0.03 radius=0.015
- added link screw_3, mass 0.002; collision cylinder length=0.03 radius=0.015; visual cylinder length=0.03 radius=0.015
- added link screw_4, mass 0.002; collision cylinder length=0.03 radius=0.015; visual cylinder length=0.03 radius=0.015
Joints:
- removed joint screw_joint
- added joint screw_joint_0: type revolute, parent box, child screw_0, origin xyz=0 0 0.486 rpy=0 0.00688 0, axis 0 0 1, limit lower=-3.14 upper=3.14 effort=1.0 velocity=1.0
- added joint screw_joint_1: type revolute, parent box, child screw_1, origin xyz=0 0.04 0.486 rpy=0 0.00688 0, axis 0 0 1, limit lower=-3.14 upper=3.14 effort=1.0 velocity=1.0
- added joint screw_joint_2: type revolute, parent box, child screw_2, origin xyz=0 0.08 0.486 rpy=0 0.00688 0, axis 0 0 1, limit lower=-3.14 upper=3.14 effort=1.0 velocity=1.0
- added joint screw_joint_3: type revolute, parent box, child screw_3, origin xyz=0 0.12 0.486 rpy=0 0.00688 0, axis 0 0 1, limit lower=-3.14 upper=3.14 effort=1.0 velocity=1.0
- added joint screw_joint_4: type revolute, parent box, child screw_4, origin xyz=0 0.16 0.486 rpy=0 0.00688 0, axis 0 0 1, limit lower=-3.14 upper=3.14 effort=1.0 velocity=1.0
