Commit message: move the screwdriver tip to the screw head

File: src/moving6/config/circu.ros2_control.xacro (robot description, xacro)
@@ -50,4 +50,11 @@
                 <state_interface name="velocity"/>
             </joint>
+            <joint name="screwdriver-screwdriver_tcp">
+                <command_interface name="position"/>
+                <state_interface name="position">
+                  <param name="initial_value">0</param>
+                </state_interface>
+                <state_interface name="velocity"/>
+            </joint>
         </ros2_control>
     </xacro:macro>

File: src/moving6/urdf/circu_robot.xacro (robot description, xacro)
@@ -162,5 +162,32 @@
   </link>
   <!-- screwdriver_tcp -->
-  <link name="screwdriver_tcp"/>
+  <link name="screwdriver_tcp">
+      <visual>
+          <geometry>
+              <cylinder length="0.03" radius="0.015"/>
+          </geometry>
+          <material name="blue">
+              <color rgba="0 0 1 1"/>
+          </material>
+      </visual>
+      <collision>
+          <geometry>
+              <cylinder length="0.03" radius="0.015"/>
+          </geometry>
+      </collision>
+      <inertial>
+          <mass value="0.002"/>
+          <inertia ixx="1e-6" iyy="1e-6" izz="1e-6" ixy="0" ixz="0" iyz="0"/>
+      </inertial>
+  </link>
+  <gazebo reference="screwdriver_tcp">
+    <sensor type="contact" name="tcp_contact">
+      <always_on>true</always_on>
+      <update_rate>50</update_rate>
+      <contact>
+        <collision>tcp_disk_collision</collision>
+      </contact>
+      </sensor>
+  </gazebo>
   <!-- cylinder and piston -->
   <link name="cylinder_link">
@@ -265,5 +292,7 @@
   </joint>
   <!-- screwdriver_tcp -->
-  <joint name="screwdriver-screwdriver_tcp" type="fixed">
+  <joint name="screwdriver-screwdriver_tcp" type="prismatic">
+    <axis xyz="0 0 1"/>
+    <limit effort="10" lower="-0.6" upper="0.0" velocity="0.1"/>
     <origin rpy="0 0 0" xyz="0.0 0.0 -0.3"/>
     <parent link="screwdriver"/>
