Commit message: fix having too many xacro files

File: src/moving6/config/circu.urdf.xacro (robot description, xacro)
@@ -3,5 +3,5 @@
     <xacro:arg name="initial_positions_file" default="initial_positions.yaml" />
     <!-- Import circu urdf file -->
-    <xacro:include filename="$(find moving6)/urdf/circu_all.xacro" />
+    <xacro:include filename="$(find moving6)/urdf/circu_robot.xacro" />
     <!-- Import control_xacro -->
     <xacro:include filename="circu.ros2_control.xacro" />

File: src/moving6/urdf/circu_robot.xacro (robot description, xacro)
@@ -2,4 +2,10 @@
 <robot name="circu_arm" xmlns:xacro="http://www.ros.org/wiki/xacro">
   <xacro:property name="prefix" value=""/>
+  <link name="world"/>
+  <joint name="base_fixed_to_world" type="fixed">
+    <parent link="world"/>
+    <child link="base_link"/>
+    <origin xyz="2 0 0" rpy="0 0 3.14"/>
+  </joint>
   <link name="base_link">
     <inertial>
@@ -171,5 +177,5 @@
           </material>
       </visual>
-      <collision>
+      <collision name="tcp_disk_collision">
           <geometry>
               <cylinder length="0.03" radius="0.015"/>
@@ -185,4 +191,5 @@
       <always_on>true</always_on>
       <update_rate>50</update_rate>
+      <topic>/contact_data</topic>
       <contact>
         <collision>tcp_disk_collision</collision>

File: src/moving6/urdf/circu_screws.urdf (robot description, URDF)
Before this commit: robot screws, 6 links, 5 joints
Links:
- added link world
Joints:
- added joint fixed: type fixed, parent world, child box, origin xyz=0 0 0.5 rpy=0 0 0
