Commit message: rename components and restructure code

File: src/unscrew_simulation/config/circu.urdf.xacro (robot description, xacro)
@@ -3,5 +3,5 @@
     <xacro:arg name="initial_positions_file" default="initial_positions.yaml" />
     <!-- Import circu urdf file -->
-    <xacro:include filename="$(find moving6)/urdf/circu_robot.xacro" />
+    <xacro:include filename="$(find unscrew_simulation)/urdf/circu_robot.xacro" />
     <!-- Import control_xacro -->
     <xacro:include filename="circu.ros2_control.xacro" />
@@ -9,5 +9,5 @@
     <gazebo>
         <plugin filename="gz_ros2_control-system" name="gz_ros2_control::GazeboSimROS2ControlPlugin">
-            <parameters>$(find moving6)/config/ros2_controllers.yaml</parameters>
+            <parameters>$(find unscrew_simulation)/config/ros2_controllers.yaml</parameters>
         </plugin>
     </gazebo>

File: src/unscrew_simulation/urdf/circu_robot.xacro (robot description, xacro)
@@ -16,10 +16,10 @@
     <visual>
       <geometry>
-        <mesh filename="package://moving6/meshes/irb6640_205/base_link.dae"/>
-      </geometry>
-    </visual>
-    <collision>
-      <geometry>
-        <mesh filename="package://moving6/meshes/irb6640_205/base_link.dae"/>
+        <mesh filename="package://unscrew_simulation/meshes/irb6640_205/base_link.dae"/>
+      </geometry>
+    </visual>
+    <collision>
+      <geometry>
+        <mesh filename="package://unscrew_simulation/meshes/irb6640_205/base_link.dae"/>
       </geometry>
     </collision>
@@ -35,5 +35,5 @@
       <origin xyz="-0.0 -0.0 -0.2345"/>
       <geometry>
-        <mesh filename="package://moving6/meshes/irb6640_205/link1.dae"/>
+        <mesh filename="package://unscrew_simulation/meshes/irb6640_205/link1.dae"/>
       </geometry>
     </visual>
@@ -41,5 +41,5 @@
       <origin xyz="-0.0 -0.0 -0.2345"/>
       <geometry>
-        <mesh filename="package://moving6/meshes/irb6640_205/link1.dae"/>
+        <mesh filename="package://unscrew_simulation/meshes/irb6640_205/link1.dae"/>
       </geometry>
     </collision>
@@ -55,5 +55,5 @@
       <origin xyz="-0.32 0.01 -0.78"/>
       <geometry>
-        <mesh filename="package://moving6/meshes/irb6640_205/link2.dae"/>
+        <mesh filename="package://unscrew_simulation/meshes/irb6640_205/link2.dae"/>
       </geometry>
     </visual>
@@ -61,5 +61,5 @@
       <origin xyz="-0.32 0.01 -0.78"/>
       <geometry>
-        <mesh filename="package://moving6/meshes/irb6640_205/link2.dae"/>
+        <mesh filename="package://unscrew_simulation/meshes/irb6640_205/link2.dae"/>
       </geometry>
     </collision>
@@ -75,5 +75,5 @@
       <origin xyz="-0.32 0.185 -2.06"/>
       <geometry>
-        <mesh filename="package://moving6/meshes/irb6640_205/link3.dae"/>
+        <mesh filename="package://unscrew_simulation/meshes/irb6640_205/link3.dae"/>
       </geometry>
     </visual>
@@ -81,5 +81,5 @@
       <origin xyz="-0.32 0.185 -2.06"/>
       <geometry>
-        <mesh filename="package://moving6/meshes/irb6640_205/link3.dae"/>
+        <mesh filename="package://unscrew_simulation/meshes/irb6640_205/link3.dae"/>
       </geometry>
     </collision>
@@ -95,5 +95,5 @@
       <origin xyz="-0.551 -8.673617379884035e-18 -2.2600000000000002"/>
       <geometry>
-        <mesh filename="package://moving6/meshes/irb6640_205/link4.dae"/>
+        <mesh filename="package://unscrew_simulation/meshes/irb6640_205/link4.dae"/>
       </geometry>
     </visual>
@@ -101,5 +101,5 @@
       <origin xyz="-0.551 -8.673617379884035e-18 -2.2600000000000002"/>
       <geometry>
-        <mesh filename="package://moving6/meshes/irb6640_205/link4.dae"/>
+        <mesh filename="package://unscrew_simulation/meshes/irb6640_205/link4.dae"/>
       </geometry>
     </collision>
@@ -115,5 +115,5 @@
       <origin xyz="-1.4625000000000001 -8.673617379884035e-18 -2.2600000000000002"/>
       <geometry>
-        <mesh filename="package://moving6/meshes/irb6640_205/link5.dae"/>
+        <mesh filename="package://unscrew_simulation/meshes/irb6640_205/link5.dae"/>
       </geometry>
     </visual>
@@ -121,5 +121,5 @@
       <origin xyz="-1.4625000000000001 -8.673617379884035e-18 -2.2600000000000002"/>
       <geometry>
-        <mesh filename="package://moving6/meshes/irb6640_205/link5.dae"/>
+        <mesh filename="package://unscrew_simulation/meshes/irb6640_205/link5.dae"/>
       </geometry>
     </collision>
@@ -135,5 +135,5 @@
       <origin xyz="-1.6625 -8.673617379884035e-18 -2.2600000000000002"/>
       <geometry>
-        <mesh filename="package://moving6/meshes/irb6640_205/link6.dae"/>
+        <mesh filename="package://unscrew_simulation/meshes/irb6640_205/link6.dae"/>
       </geometry>
     </visual>
@@ -141,5 +141,5 @@
       <origin xyz="-1.6625 -8.673617379884035e-18 -2.2600000000000002"/>
       <geometry>
-        <mesh filename="package://moving6/meshes/irb6640_205/link6.dae"/>
+        <mesh filename="package://unscrew_simulation/meshes/irb6640_205/link6.dae"/>
       </geometry>
     </collision>
@@ -157,5 +157,5 @@
       <origin xyz="0.0 0.0 0.0" rpy="-1.5707963267948966 -1.5707963267948966 0"/>
       <geometry>
-        <mesh filename="package://moving6/meshes/screwdriver/weber_screwdriver_sevp30_with_tx10bit.dae"/>
+        <mesh filename="package://unscrew_simulation/meshes/screwdriver/weber_screwdriver_sevp30_with_tx10bit.dae"/>
       </geometry>
     </visual>
@@ -163,5 +163,5 @@
       <origin xyz="0.0 0.0 0.0" rpy="-1.5707963267948966 -1.5707963267948966 0"/>
       <geometry>
-        <mesh filename="package://moving6/meshes/screwdriver/weber_screwdriver_sevp30_with_tx10bit.dae"/>
+        <mesh filename="package://unscrew_simulation/meshes/screwdriver/weber_screwdriver_sevp30_with_tx10bit.dae"/>
       </geometry>
     </collision>
@@ -207,5 +207,5 @@
       <origin xyz="0.3647 -0.0 -0.6345000000000001"/>
       <geometry>
-        <mesh filename="package://moving6/meshes/irb6640_205/cylinder_link.dae"/>
+        <mesh filename="package://unscrew_simulation/meshes/irb6640_205/cylinder_link.dae"/>
       </geometry>
     </visual>
@@ -213,5 +213,5 @@
       <origin xyz="0.3647 -0.0 -0.6345000000000001"/>
       <geometry>
-        <mesh filename="package://moving6/meshes/irb6640_205/cylinder_link.dae"/>
+        <mesh filename="package://unscrew_simulation/meshes/irb6640_205/cylinder_link.dae"/>
       </geometry>
     </collision>
@@ -226,5 +226,5 @@
       <origin xyz="-0.10005 0.01 -0.71275"/>
       <geometry>
-        <mesh filename="package://moving6/meshes/irb6640_205/piston_link.dae"/>
+        <mesh filename="package://unscrew_simulation/meshes/irb6640_205/piston_link.dae"/>
       </geometry>
     </visual>
@@ -232,5 +232,5 @@
       <origin xyz="-0.10005 0.01 -0.71275"/>
       <geometry>
-        <mesh filename="package://moving6/meshes/irb6640_205/piston_link.dae"/>
+        <mesh filename="package://unscrew_simulation/meshes/irb6640_205/piston_link.dae"/>
       </geometry>
     </collision>
